File: hall.kicad_sch (KiCad schematic)
At the start: 5 parts, among them U5 SS49E

Commit message: schematic: Some changes
* Add test points for hall sensors
* Assign 2.54 mm header footprints
* Fix CAN termination resistor
Parts:
- U6: renamed from U5; footprint (none) -> Package_TO_SOT_THT:TO-92_Inline
- renumbered C17 to C19, C18 to C20, R9 to R11, R10 to R12
Changed lines of the file:
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@@
 		(on_board yes)
 		(dnp no)
-		(property "Reference" "C18"
+		(property "Reference" "C20"
 			(at 172.72 95.2562 0)
 			(effects
@@
 		(dnp no)
 		(fields_autoplaced yes)
-		(property "Reference" "R9"
+		(property "Reference" "R11"
 			(at 167.64 85.09 90)
 			(effects
@@
 		(dnp no)
 		(fields_autoplaced yes)
-		(property "Reference" "#PWR028"
+		(property "Reference" "#PWR029"
 			(at 175.26 106.68 0)
 			(effects
@@
 		(dnp no)
 		(fields_autoplaced yes)
-		(property "Reference" "#PWR024"
+		(property "Reference" "#PWR025"
 			(at 130.81 100.33 0)
 			(effects
@@
 		(on_board yes)
 		(dnp no)
-		(property "Reference" "R10"
+		(property "Reference" "R12"
 			(at 185.42 95.2499 0)
 			(effects
@@
 		(dnp no)
 		(fields_autoplaced yes)
-		(property "Reference" "#PWR026"
+		(property "Reference" "#PWR027"
 			(at 182.88 106.68 0)
 			(effects
@@
 		(on_board yes)
 		(dnp no)
-		(property "Reference" "#PWR022"
+		(property "Reference" "#PWR023"
 			(at 130.81 90.17 0)
 			(effects
@@
 		(dnp no)
 		(fields_autoplaced yes)
-		(property "Reference" "#PWR020"
+		(property "Reference" "#PWR021"
 			(at 151.13 107.95 0)
 			(effects
@@
 		(dnp no)
 		(fields_autoplaced yes)
-		(property "Reference" "U5"
+		(property "Reference" "U6"
 			(at 147.32 88.8999 0)
 			(effects
@@
 			)
 		)
-		(property "Footprint" ""
+		(property "Footprint" "Package_TO_SOT_THT:TO-92_Inline"
 			(at 153.67 90.17 0)
 			(effects
@@
 		(on_board yes)
 		(dnp no)
-		(property "Reference" "#PWR018"
+		(property "Reference" "#PWR019"
 			(at 151.13 82.55 0)
 			(effects
@@
 		(on_board yes)
 		(dnp no)
-		(property "Reference" "C17"
+		(property "Reference" "C19"
 			(at 128.27 88.9062 0)
 			(effects

Commit message: Changed SS49E footprint and updated to KiCAD 9
Parts:
- U5: renamed from U6; footprint Package_TO_SOT_THT:TO-92_Inline -> SS49E:SS49E_TO_92_Inline
- renumbered C19 to C17, C20 to C18, R12 to R10, R11 to R9
Changed lines of the file:
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@@
 (kicad_sch
-	(version 20231120)
+	(version 20250114)
 	(generator "eeschema")
-	(generator_version "8.0")
+	(generator_version "9.0")
 	(paper "A4")
 	(junction
@@
 		(shape output)
 		(at 187.96 90.17 0)
-		(fields_autoplaced yes)
 		(effects
 			(font
@@
 		(on_board yes)
 		(dnp no)
-		(property "Reference" "C20"
+		(property "Reference" "C18"
 			(at 172.72 95.2562 0)
 			(effects
@@
 		(dnp no)
 		(fields_autoplaced yes)
-		(property "Reference" "R11"
+		(property "Reference" "R9"
 			(at 167.64 85.09 90)
 			(effects
@@
 		(dnp no)
 		(fields_autoplaced yes)
-		(property "Reference" "#PWR029"
+		(property "Reference" "#PWR028"
 			(at 175.26 106.68 0)
 			(effects
@@
 		(dnp no)
 		(fields_autoplaced yes)
-		(property "Reference" "#PWR025"
+		(property "Reference" "#PWR024"
 			(at 130.81 100.33 0)
 			(effects
@@
 		(on_board yes)
 		(dnp no)
-		(property "Reference" "R12"
+		(property "Reference" "R10"
 			(at 185.42 95.2499 0)
 			(effects
@@
 		(dnp no)
 		(fields_autoplaced yes)
-		(property "Reference" "#PWR027"
+		(property "Reference" "#PWR026"
 			(at 182.88 106.68 0)
 			(effects
@@
 		(on_board yes)
 		(dnp no)
-		(property "Reference" "#PWR023"
+		(property "Reference" "#PWR022"
 			(at 130.81 90.17 0)
 			(effects
@@
 		(dnp no)
 		(fields_autoplaced yes)
-		(property "Reference" "#PWR021"
+		(property "Reference" "#PWR020"
 			(at 151.13 107.95 0)
 			(effects
@@
 		(dnp no)
 		(fields_autoplaced yes)
-		(property "Reference" "U6"
+		(property "Reference" "U5"
 			(at 147.32 88.8999 0)
 			(effects
@@
 			)
 		)
-		(property "Footprint" "Package_TO_SOT_THT:TO-92_Inline"
+		(property "Footprint" "SS49E:SS49E_TO_92_Inline"
 			(at 153.67 90.17 0)
 			(effects
@@
 		(on_board yes)
 		(dnp no)
-		(property "Reference" "#PWR019"
+		(property "Reference" "#PWR018"
 			(at 151.13 82.55 0)
 			(effects
@@
 		(on_board yes)
 		(dnp no)
-		(property "Reference" "C19"
+		(property "Reference" "C17"
 			(at 128.27 88.9062 0)
 			(effects
